Commit message: added reach7 URDF

File: ROS/reach_system_one_support/urdf/reach5mini.urdf (robot description, URDF)
Before this commit: robot reach5mini, 8 links, 7 joints
Links:
- link base_link: geometry collision cylinder length=0.150 radius=0.020; visual mesh filename=package://reach_system_one_support/meshes/reach5mini/visual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
- link forearm_link: geometry collision cylinder length=0.040 radius=0.020; visual mesh filename=package://reach_system_one_support/meshes/reach5mini/visual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
- link jaw1: geometry collision box size=0.03 0.09 0.01; visual mesh filename=package://reach_system_one_support/meshes/reach5mini/visual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
- link jaw2: geometry collision box size=0.03 0.09 0.01; visual mesh filename=package://reach_system_one_support/meshes/reach5mini/visual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
- link shoulder_link: geometry collision cylinder length=0.066 radius=0.020; visual mesh filename=package://reach_system_one_support/meshes/reach5mini/visual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
- link upper_arm_link: geometry collision cylinder length=0.040 radius=0.020; collision cylinder length=0.145 radius=0.020
- link wrist_link: geometry collision cylinder length=0.140 radius=0.020; visual mesh filename=package://reach_system_one_support/meshes/reach5mini/visual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
