Commit message: updated bravo urdf

File: ROS/bravo_description/urdf/bravo_5S.urdf (robot description, URDF)
Before this commit: robot bravo7, 13 links, 12 joints
Links:
- removed link bravo_rs2_161_link
- removed link bravo_rs2_214_link
- removed link bravo_rs2_250_212_214_link
- added link bravo_RS2-1013_base_link; visual mesh filename=package://bravo_description/meshes/RS2-1013_base.stl
- added link bravo_RS2-1026_base_link; visual mesh filename=package://bravo_description/meshes/RS2-1026_0_base.stl
- added link bravo_RS2-1030_base_link; visual mesh filename=package://bravo_description/meshes/RS2-1030.stl
Joints:
- removed joint bravo_axis_f
- removed joint bravo_axis_g
- added joint bravo_rs2_313_joint: type fixed, parent bravo_RS2-1013_base_link, child bravo_RS2-1030_base_link, origin rpy=0 0 0
- added joint bravo_rs2_326_joint: type fixed, parent bravo_RS2-1030_base_link, child bravo_RS2-1026_base_link, origin xyz=0 0 0 rpy=0 0 0
- joint bravo_axis_b: origin xyz=-0.0408 0 -0.08863 rpy=0 3.14159 0 -> xyz=0.0408 0 0.09645 rpy=0 0 0; parent bravo_rs2_161_link -> bravo_rs2_268_link
- joint bravo_axis_c: child bravo_rs2_161_link -> bravo_rs2_268_link; origin xyz=-0.0408 0 0.063 rpy=0 0 0 -> xyz=-0.0868 0 -0.29355 rpy=0 0 3.1415; parent bravo_rs2_214_link -> bravo_RS2-1013_base_link
- joint bravo_axis_d: axis 0 0 -1 -> 0 1 0; child bravo_rs2_214_link -> bravo_RS2-1013_base_link; limit lower=0.0 upper=6.3 effort=9.0 velocity=0.5 -> lower=0.0 upper=3.5 effort=9.0 velocity=0.5; origin xyz=0.0408 0 0.09695 rpy=0 0 3.14159 -> xyz=-0.046 0 0.0674 rpy=0 0 0; parent bravo_rs2_268_link -> bravo_rs2_217_link
- joint bravo_axis_e: axis 0 1 0 -> 0 0 -1; child bravo_rs2_268_link -> bravo_rs2_217_link; limit lower=0.0 upper=3.5 effort=9.0 velocity=0.5 -> lower=0.0 upper=6.3 effort=9.0 velocity=0.5; origin xyz=-0.0052 0 -0.29055 rpy=0 0 0 -> xyz=0.0665 0 0.078 rpy=0 0 0; parent bravo_rs2_250_212_214_link -> bravo_rs2_266_link

File: ROS/bravo_description/urdf/bravo_7C.urdf (robot description, URDF)
Before this commit: robot bravo5, 11 links, 10 joints
Links:
- added link bravo_rs2_161_link; visual mesh filename=package://bravo_description/meshes/RS2-161.stl
- added link bravo_rs2_214_link; visual mesh filename=package://bravo_description/meshes/RS2-214.stl
Joints:
- added joint bravo_axis_f: type revolute, parent bravo_rs2_217_link, child bravo_rs2_250_212_214_link, origin xyz=-0.046 0 0.0674 rpy=0 0 0, axis 0 1 0, limit lower=0.0 upper=3.5 effort=9.0 velocity=0.5
- added joint bravo_axis_g: type revolute, parent bravo_rs2_266_link, child bravo_rs2_217_link, origin xyz=0.0665 0 0.078 rpy=0 0 0, axis 0 0 -1, limit lower=0.0 upper=6.3 effort=9.0 velocity=0.5
- joint bravo_axis_b: axis 0 0 1 -> 0 0 -1; origin xyz=0.0408 0 0.09645 rpy=0 0 0 -> xyz=-0.0408 0 -0.08863 rpy=0 3.14159 0; parent bravo_rs2_268_link -> bravo_rs2_161_link
- joint bravo_axis_c: child bravo_rs2_268_link -> bravo_rs2_161_link; origin xyz=-0.0052 0 -0.29055 rpy=0 0 0 -> xyz=-0.0408 0 0.063 rpy=0 0 0; parent bravo_rs2_250_212_214_link -> bravo_rs2_214_link
- joint bravo_axis_d: axis 0 1 0 -> 0 0 -1; child bravo_rs2_250_212_214_link -> bravo_rs2_214_link; limit lower=0.0 upper=3.5 effort=9.0 velocity=0.5 -> lower=0.0 upper=6.3 effort=9.0 velocity=0.5; origin xyz=-0.046 0 0.0674 rpy=0 0 0 -> xyz=0.0408 0 0.09695 rpy=0 0 3.14159; parent bravo_rs2_217_link -> bravo_rs2_268_link
- joint bravo_axis_e: axis 0 0 1 -> 0 1 0; child bravo_rs2_217_link -> bravo_rs2_268_link; limit lower=0.0 upper=6.3 effort=9.0 velocity=0.5 -> lower=0.0 upper=3.5 effort=9.0 velocity=0.5; origin xyz=0.0665 0 0.078 rpy=0 0 0 -> xyz=-0.0052 0 -0.29355 rpy=0 0 0; parent bravo_rs2_266_link -> bravo_rs2_250_212_214_link
