Commit message: Updated alpha_5.urdf.xacro, standard_jaws.urdf.xacro, and 38 more files...
Added Alpha 5 Collision meshes
Added bpl_bravo_description package
-  Bravo 7 and Bravo 5 Urdf with collision
Updated documentation for bpl_bravo_description

File: ROS/bpl_alpha_description/urdf/alpha_5.urdf.xacro (robot description, xacro)
@@ -1,5 +1,5 @@
 <?xml version="1.0"?>
 <robot name="alpha_5" xmlns:xacro="http://ros.org/wiki/xacro">
-    <xacro:macro name="alpha_5" params="parent *origin name:=alpha5">
+    <xacro:macro name="alpha_5" params="parent *origin name:=alpha_5">
         <joint name="${name}_joint" type="fixed">
             <xacro:insert_block name="origin" />
@@ -20,4 +20,10 @@
                 <material name="alpha_black"/>
             </visual>
+            <collision>
+                <geometry>
+                    <cylinder length="0.150" radius="0.020" />
+                </geometry>
+                <origin rpy="0 1.57075 0" xyz="-0.075 0 0" />
+            </collision>
         </link>
         <joint name="${name}_base_link_joint" type="fixed">
@@ -34,4 +40,10 @@
                 <material name="${name}_black"/>
             </visual>
+            <collision>
+                <geometry>
+                    <cylinder length="0.066" radius="0.020" />
+                </geometry>
+                <origin rpy="0 0 0" xyz="0 0 0.000" />
+            </collision>
         </link>
         <joint name="${name}_axis_e" type="revolute">
@@ -50,4 +62,22 @@
                 <material name="${name}_black"/>
             </visual>
+            <collision>
+                <geometry>
+                    <cylinder length="0.145" radius="0.020" />
+                </geometry>
+                <origin rpy="0 0 0" xyz="-0.02 0 -0.0725" />
+            </collision>
+            <collision>
+                <geometry>
+                    <cylinder length="0.040" radius="0.020" />
+                </geometry>
+                <origin rpy="1.5707 0 0" xyz="0 0 0" />
+            </collision>
+            <collision>
+                <geometry>
+                    <cylinder length="0.040" radius="0.020" />
+                </geometry>
+                <origin rpy="1.5707 0 0" xyz="-0.040 0 -0.1453" />
+            </collision>
         </link>
         <joint name="${name}_axis_d" type="revolute">
@@ -66,4 +96,10 @@
                 <material name="${name}_black"/>
             </visual>
+            <collision>
+                <geometry>
+                    <cylinder length="0.033" radius="0.020" />
+                </geometry>
+                <origin rpy="0 0 0" xyz="0.02 0 0.0165" />
+            </collision>
         </link>
         <joint name="${name}_axis_c" type="revolute">
@@ -82,4 +118,10 @@
                 <material name="${name}_black"/>
             </visual>
+            <collision>
+                <geometry>
+                    <cylinder length="0.10975" radius="0.020" />
+                </geometry>
+                <origin rpy="0 0 0" xyz="0.00 0 0.054875" />
+            </collision>
         </link>
             <joint name="${name}_axis_b" type="revolute">

File: ROS/bpl_alpha_description/urdf/end_effectors/standard_jaws.urdf.xacro (robot description, xacro)
@@ -12,19 +12,25 @@
         </joint>
         <link name="${name}_base_link">
-          <visual>
-            <geometry>
-              <mesh filename="package://bpl_alpha_description/meshes/end_effectors/RS1-124.stl"/>
-            </geometry>
-            <material name="${name}_black"/>
-          </visual>
+            <visual>
+                <geometry>
+                    <mesh filename="package://bpl_alpha_description/meshes/end_effectors/RS1-124.stl"/>
+                </geometry>
+                <material name="${name}_black"/>
+            </visual>
         </link>
         <link name="${name}_rs1_130_link">
-          <visual>
-            <geometry>
-              <mesh filename="package://bpl_alpha_description/meshes/end_effectors/RS1-130.stl"/>
-            </geometry>
-            <material name="${name}_black"/>
-            <origin xyz="0 0 0" rpy="0 0 0"/>
-          </visual>
+            <visual>
+                <geometry>
+                    <mesh filename="package://bpl_alpha_description/meshes/end_effectors/RS1-130.stl"/>
+                </geometry>
+                <material name="${name}_black"/>
+                <origin xyz="0 0 0" rpy="0 0 0"/>
+            </visual>
+            <collision>
+                <geometry>
+                    <box size="0.012 0.03 0.09"/>
+                </geometry>
+                <origin xyz="0.0 -0.008 0.045" rpy="0 0 0"/>
+            </collision>
         </link>
         <joint name="${name}_rs1_130_joint" type="revolute">
@@ -37,11 +43,17 @@
         </joint>
         <link name="${name}_rs1_139_link">
-          <visual>
-            <geometry>
-              <mesh filename="package://bpl_alpha_description/meshes/end_effectors/RS1-139.stl"/>
-            </geometry>
-            <material name="${name}_black"/>
-            <origin xyz="0 0 0" rpy="0 0 0"/>
-          </visual>
+            <visual>
+                <geometry>
+                    <mesh filename="package://bpl_alpha_description/meshes/end_effectors/RS1-139.stl"/>
+                </geometry>
+                <material name="${name}_black"/>
+                <origin xyz="0 0 0" rpy="0 0 0"/>
+            </visual>
+            <collision>
+                <geometry>
+                    <box size="0.012 0.03 0.09"/>
+                </geometry>
+                <origin xyz="0.0 0.008 0.045" rpy="0 0 0"/>
+            </collision>
         </link>
         <joint name="${name}_rs1_139_joint" type="revolute">
