Commit message: Changed bravo config

File: ROS/bpl_bravo_description/urdf/bravo_5.urdf.xacro (robot description, xacro)
@@ -186,5 +186,5 @@
         <joint name="${name}_1023_1_end_joint" type="fixed">
             <parent link="${name}_1023_1_joint_link"/>
-            <origin xyz="0 0 0.0056" rpy="0 0 -1.5707"/>
+            <origin xyz="0 0 0.0056" rpy="0 0 0"/>
             <child link="${name}_1023_1_end_link"/>
         </joint>

File: ROS/bpl_bravo_description/urdf/bravo_5_example.urdf (robot description, URDF)
Before this commit: robot bravo_5_example, 20 links, 19 joints
Joints:
- joint bravo_1023_1_end_joint: origin xyz=0 0 0.0056 rpy=0 0 -1.5707 -> xyz=0 0 0.0056 rpy=0 0 0

File: ROS/bpl_bravo_description/urdf/bravo_7.urdf.xacro (robot description, xacro)
@@ -273,5 +273,5 @@
         <joint name="${name}_1023_1_end_joint" type="fixed">
             <parent link="${name}_1023_1_joint_link"/>
-            <origin xyz="0 0 0.0056" rpy="0 0 -1.5707"/>
+            <origin xyz="0 0 0.0056" rpy="0 0 0"/>
             <child link="${name}_1023_1_end_link"/>
         </joint>

File: ROS/bpl_bravo_description/urdf/bravo_7_example.urdf (robot description, URDF)
Before this commit: robot bravo_7_example, 26 links, 25 joints
Joints:
- joint bravo_1023_1_end_joint: origin xyz=0 0 0.0056 rpy=0 0 -1.5707 -> xyz=0 0 0.0056 rpy=0 0 0
