Commit message: Modified bravo_7 urdf to remove hard-coded bravo_black reference. Added new xacro and launch file for two bravo 7s at once

File: ROS2/bpl_bravo_description/urdf/bravo_7.urdf.xacro (robot description, xacro)
@@ -8,5 +8,5 @@
             <origin xyz="0 0 0" rpy="0 0 0"/>
         </joint>
-        <material name="bravo_black">
+        <material name="${name}_black">
             <color rgba="0.3 0.3 0.3 1"/>
         </material>
@@ -16,5 +16,5 @@
                     <mesh filename="package://bpl_bravo_description/meshes/RS2-1019_base.stl"/>
                 </geometry>
-                <material name="bravo_black"/>
+                <material name="${name}_black"/>
             </visual>
            <collision>
@@ -49,5 +49,5 @@
                     <mesh filename="package://bpl_bravo_description/meshes/RS2-1019_end.stl"/>
                 </geometry>
-                <material name="bravo_black"/>
+                <material name="${name}_black"/>
             </visual>
         </link>
@@ -62,5 +62,5 @@
                     <mesh filename="package://bpl_bravo_description/meshes/RS2-1013_base.stl"/>
                 </geometry>
-                <material name="bravo_black"/>
+                <material name="${name}_black"/>
             </visual>
             <collision>
@@ -89,5 +89,5 @@
                     <mesh filename="package://bpl_bravo_description/meshes/RS2-1013_end.stl"/>
                 </geometry>
-                <material name="bravo_black"/>
+                <material name="${name}_black"/>
             </visual>
             <collision>
@@ -114,5 +114,5 @@
                     <mesh filename="package://bpl_bravo_description/meshes/RS2-1026_0_base.stl"/>
                 </geometry>
-                <material name="bravo_black"/>
+                <material name="${name}_black"/>
             </visual>
             <collision>
@@ -141,5 +141,5 @@
                     <mesh filename="package://bpl_bravo_description/meshes/RS2-1026_0_end.stl"/>
                 </geometry>
-                <material name="bravo_black"/>
+                <material name="${name}_black"/>
             </visual>
             <collision>
@@ -175,5 +175,5 @@
                     <mesh filename="package://bpl_bravo_description/meshes/RS2-1026_1_end.stl"/>
                 </geometry>
-                <material name="bravo_black"/>
+                <material name="${name}_black"/>
                 <origin xyz="0 0 0 " rpy="0 0 3.14159"/>
             </visual>
@@ -201,5 +201,5 @@
                     <mesh filename="package://bpl_bravo_description/meshes/RS2-1023_0_base.stl"/>
                 </geometry>
-                <material name="bravo_black"/>
+                <material name="${name}_black"/>
             </visual>
             <collision>
@@ -228,5 +228,5 @@
                     <mesh filename="package://bpl_bravo_description/meshes/RS2-1023_0_end.stl"/>
                 </geometry>
-                <material name="bravo_black"/>
+                <material name="${name}_black"/>
             </visual>
             <collision>
@@ -262,5 +262,5 @@
                     <mesh filename="package://bpl_bravo_description/meshes/RS2-1023_1_end.stl"/>
                 </geometry>
-                <material name="bravo_black"/>
+                <material name="${name}_black"/>
             </visual>
             <collision>
@@ -287,5 +287,5 @@
                     <mesh filename="package://bpl_bravo_description/meshes/RS2-1028.stl"/>
                 </geometry>
-                <material name="bravo_black"/>
+                <material name="${name}_black"/>
             </visual>
             <collision>
@@ -328,5 +328,5 @@
                     <mesh filename="package://bpl_bravo_description/meshes/RS2-1030.stl"/>
                 </geometry>
-                <material name="bravo_black"/>
+                <material name="${name}_black"/>
             </visual>
             <collision>
