Commit message: Modified Bravo 5 urdf to remove hard coded reference. Updated and rename double bravo launch and xarco files

File: ROS2/bpl_bravo_description/urdf/bravo_5.urdf.xacro (robot description, xacro)
@@ -8,5 +8,5 @@
             <origin xyz="0 0 0" rpy="0 0 0"/>
         </joint>
-        <material name="bravo_black">
+        <material name="${name}_black">
             <color rgba="0.3 0.3 0.3 1"/>
         </material>
@@ -16,5 +16,5 @@
                     <mesh filename="package://bpl_bravo_description/meshes/RS2-1019_base.stl"/>
                 </geometry>
-                <material name="bravo_black"/>
+                <material name="${name}_black"/>
             </visual>
            <collision>
@@ -49,5 +49,5 @@
                     <mesh filename="package://bpl_bravo_description/meshes/RS2-1019_end.stl"/>
                 </geometry>
-                <material name="bravo_black"/>
+                <material name="${name}_black"/>
             </visual>
         </link>
@@ -62,5 +62,5 @@
                     <mesh filename="package://bpl_bravo_description/meshes/RS2-1013_base.stl"/>
                 </geometry>
-                <material name="bravo_black"/>
+                <material name="${name}_black"/>
             </visual>
             <collision>
@@ -89,5 +89,5 @@
                     <mesh filename="package://bpl_bravo_description/meshes/RS2-1013_end.stl"/>
                 </geometry>
-                <material name="bravo_black"/>
+                <material name="${name}_black"/>
             </visual>
             <collision>
@@ -114,5 +114,5 @@
                     <mesh filename="package://bpl_bravo_description/meshes/RS2-1023_0_base.stl"/>
                 </geometry>
-                <material name="bravo_black"/>
+                <material name="${name}_black"/>
             </visual>
             <collision>
@@ -141,5 +141,5 @@
                     <mesh filename="package://bpl_bravo_description/meshes/RS2-1023_0_end.stl"/>
                 </geometry>
-                <material name="bravo_black"/>
+                <material name="${name}_black"/>
             </visual>
             <collision>
@@ -175,5 +175,5 @@
                     <mesh filename="package://bpl_bravo_description/meshes/RS2-1023_1_end.stl"/>
                 </geometry>
-                <material name="bravo_black"/>
+                <material name="${name}_black"/>
             </visual>
             <collision>
@@ -200,5 +200,5 @@
                     <mesh filename="package://bpl_bravo_description/meshes/RS2-1028.stl"/>
                 </geometry>
-                <material name="bravo_black"/>
+                <material name="${name}_black"/>
             </visual>
             <collision>
@@ -241,5 +241,5 @@
                     <mesh filename="package://bpl_bravo_description/meshes/RS2-1030.stl"/>
                 </geometry>
-                <material name="bravo_black"/>
+                <material name="${name}_black"/>
             </visual>
             <collision>

File: ROS2/bpl_bravo_description/urdf/bravo_double_example.urdf.xacro (robot description, xacro)
@@ -6,6 +6,7 @@
       <origin xyz="0 0 0" rpy="0 0 0"/>
     </xacro:bravo_7>
-    <xacro:bravo_7 parent="base_link" name="bravo_b">
+  <xacro:include filename="$(find bpl_bravo_description)/urdf/bravo_5.urdf.xacro"/>
+    <xacro:bravo_5 parent="base_link" name="bravo_b">
       <origin xyz="0.635 0 0" rpy="0 0 0"/>
-    </xacro:bravo_7>
+    </xacro:bravo_5>
 </robot>
