Commit message: double_bravo

File: ROS2/bpl_bravo_description/urdf/bravo_double_example.urdf.xacro (robot description, xacro)
@@ -4,9 +4,9 @@
     <link name="base_link"/>
     <xacro:bravo_7 parent="base_link" name="bravo_a">
-      <origin xyz="0 0 0" rpy="0 0 0"/>
+      <origin xyz="0.635 0 0" rpy="0 0 0"/>
     </xacro:bravo_7>
   <xacro:include filename="$(find bpl_bravo_description)/urdf/bravo_5.urdf.xacro"/>
     <xacro:bravo_5 parent="base_link" name="bravo_b">
-      <origin xyz="0.635 0 0" rpy="0 0 0"/>
+      <origin xyz="0 0 0" rpy="0 0 0"/>
     </xacro:bravo_5>
 </robot>

Commit message: final_demo

File: ROS2/bpl_bravo_description/urdf/bravo_double_example.urdf.xacro (robot description, xacro)
@@ -4,5 +4,5 @@
     <link name="base_link"/>
     <xacro:bravo_7 parent="base_link" name="bravo_a">
-      <origin xyz="0.635 0 0" rpy="0 0 0"/>
+      <origin xyz="0.430 0 0" rpy="0 0 0"/>
     </xacro:bravo_7>
   <xacro:include filename="$(find bpl_bravo_description)/urdf/bravo_5.urdf.xacro"/>
