Commit message: mk2_visualsiation_fix

File: ROS/bpl_bravo_description_mk2/urdf/bravo_5_example.urdf (robot description, URDF)
Before this commit: robot bravo_5_example, 20 links, 19 joints
Links:
- link bravo_1023_0_base_link: geometry collision cylinder length=0.059 radius=0.0408; collision cylinder length=0.0599 radius=0.0408
- link bravo_1023_0_joint_link: geometry collision cylinder length=0.02335 radius=0.0408; collision cylinder length=0.0851 radius=0.0408
- link bravo_1023_1_joint_link: geometry collision cylinder length=0.003 radius=0.0408; visual mesh filename=package://bpl_bravo_description_mk2/meshes/RS2-1023-C.stl
Joints:
- joint bravo_1023_0_end_joint: origin xyz=0.0408 0 -0.0956 rpy=3.14159 0 0 -> xyz=0.0408 0 -0.08705 rpy=3.14159 0 0

File: ROS/bpl_bravo_description_mk2/urdf/bravo_7_example.urdf (robot description, URDF)
Before this commit: robot bravo_7_example, 26 links, 25 joints
Links:
- link bravo_1023_0_base_link: geometry collision cylinder length=0.059 radius=0.0408; collision cylinder length=0.0599 radius=0.0408
- link bravo_1023_0_joint_link: geometry collision cylinder length=0.02335 radius=0.0408; collision cylinder length=0.0851 radius=0.0408
- link bravo_1023_1_joint_link: geometry collision cylinder length=0.003 radius=0.0408; visual mesh filename=package://bpl_bravo_description_mk2/meshes/RS2-1023-C.stl
- link bravo_1026_0_base_link: geometry collision cylinder length=0.059 radius=0.0408; collision cylinder length=0.0599 radius=0.0408
- link bravo_1026_0_joint_link: geometry collision cylinder length=0.02335 radius=0.0408; collision cylinder length=0.0851 radius=0.0408
- link bravo_1026_1_joint_link: geometry collision cylinder length=0.003 radius=0.0408; visual mesh filename=package://bpl_bravo_description_mk2/meshes/RS2-1026-C.stl
Joints:
- joint bravo_1023_0_end_joint: origin xyz=0.0408 0 -0.0956 rpy=3.14159 0 0 -> xyz=0.0408 0 -0.08705 rpy=3.14159 0 0
- joint bravo_1026_0_end_joint: origin xyz=0.0408 0 -0.0956 rpy=3.14159 0 0 -> xyz=0.0408 0 -0.08705 rpy=3.14159 0 0
